Commit message: kinect was added to the the existing pioneer model, ros plugins were added to the gazebo model for funcionality

File: p3dx_description/urdf/pioneer3dx.xacro (robot description, xacro)
@@ -223,3 +223,89 @@
 		<child link="lms100" />
 	</joint>
+<!-- kinect sensor -->
+	<joint name="kinect_joint" type="fixed">
+		<origin rpy="0 0 0" xyz="0.109 0 0.509" />
+		<parent link="base_link" />
+		<child link="kinect_link" />
+	</joint>
+<!-- SENSOR -->
+  <link name="kinect_link">
+        <inertial>
+           <mass value="0.1"/>
+           <origin xyz="0 0 0" />
+           <inertia ixx="1" ixy="0" ixz="0" iyy="1" iyz="0" izz="1" />
+        </inertial>
+        <collision name="collision">
+           <geometry>
+             <box size = "0.073000 0.276000 0.072000"/>
+           </geometry>
+        </collision>
+        <visual name="visual">
+           <geometry>
+              <mesh filename="model://kinect/meshes/kinect.dae"/>
+           </geometry>
+        </visual>
+</link>
+<!--    <link name="kinect_link">
+        <inertial>
+           <mass value="0.1"/>
+           <origin xyz="0 0 0" />
+           <inertia ixx="1" ixy="0" ixz="0" iyy="1" iyz="0" izz="1" />
+        </inertial>
+        <collision name="collision">
+           <geometry>
+             <box size = "0.073000 0.276000 0.072000"/>
+           </geometry>
+        </collision>
+        <visual name="visual">
+           <geometry>
+              <mesh filename="model://kinect/meshes/kinect.dae"/>
+           </geometry>
+        </visual>
+      <sensor name="camera" type="depth">
+        <update_rate>20</update_rate>
+        <camera>
+          <horizontal_fov>1.047198</horizontal_fov>
+          <image>
+            <width>640</width>
+            <height>480</height>
+            <format>R8G8B8</format>
+          </image>
+          <clip>
+            <near>0.05</near>
+            <far>3</far>
+          </clip>
+        </camera>
+      </sensor>
+    </link>
+	<joint name="base_front_top_joint" type="fixed">
+		<origin rpy="0 0 0" xyz="0.109 0 0.509" />
+		<parent link="base_link" />
+		<child link="kinect_link" />
+	</joint>
+<gazebo reference="kinect_link">
+    <plugin name="kinect_link_controller" filename="libgazebo_ros_openni_kinect.so">
+       <baseline>0.2</baseline>
+       <alwaysOn>true</alwaysOn>
+       <updateRate>1.0</updateRate>
+       <cameraName>camera_ir</cameraName>
+       <imageTopicName>camera/depth/image_raw</imageTopicName>
+       <cameraInfoTopicName>/camera/depth/camera_info</cameraInfoTopicName>
+       <depthImageTopicName>/camera/depth/image_raw</depthImageTopicName>
+       <depthImageInfoTopicName>camera/depth/camera_info</depthImageInfoTopicName>
+       <pointCloudTopicName>camera/depth/points</pointCloudTopicName>
+       <frameName>kinetic_link</frameName>
+       <pointCloudCutoff>0.5</pointCloudCutoff>
+       <distortionK1>0.00000001</distortionK1>
+       <distortionK2>0.00000001</distortionK2>
+       <distortionK3>0.00000001</distortionK3>
+       <distortionT1>0.00000001</distortionT1>
+       <distortionT2>0.00000001</distortionT2>
+       <CxPrime>0</CxPrime>
+       <Cx>0</Cx>
+       <Cy>0</Cy>
+       <focalLength>0</focalLength>
+       <hackBaseline>0</hackBaseline>
+    </plugin>
+</gazebo-->
 </robot>
